File: mainboard/apple1.kicad_pcb (KiCad board)
At the start: 2 copper layers, 393.7 x 228.6 mm, 6 parts

Commit message: Further work on the schematics/file organization
Parts:
- added A1: MMI6301, Package_DIP:DIP-16_W7.62mm, F.Cu at (39.7, 289.0)
- added A11: MK4096, Package_DIP:DIP-16_W7.62mm, F.Cu at (245.6, 347.5)
- added A12: MK4096, Package_DIP:DIP-16_W7.62mm, F.Cu at (256.4, 347.5)
- added A13: MK4096, Package_DIP:DIP-16_W7.62mm, F.Cu at (267.1, 347.5)
- added A14: MK4096, Package_DIP:DIP-16_W7.62mm, F.Cu at (277.9, 347.5)
- added A15: MK4096, Package_DIP:DIP-16_W7.62mm, F.Cu at (307.9, 351.8)
- added A16: MK4096, Package_DIP:DIP-16_W7.62mm, F.Cu at (288.7, 347.5)
- added A17: MK4096, Package_DIP:DIP-16_W7.62mm, F.Cu at (245.6, 369.4)
- added A18: MK4096, Package_DIP:DIP-16_W7.62mm, F.Cu at (256.4, 369.4)
- added A2: MMI6301, Package_DIP:DIP-16_W7.62mm, F.Cu at (51.0, 289.0)
- added B1: 7400, Package_DIP:DIP-14_W7.62mm, F.Cu at (489.6, 275.6)
- added B11: MK4096, Package_DIP:DIP-16_W7.62mm, F.Cu at (267.1, 369.4)
- added B12: MK4096, Package_DIP:DIP-16_W7.62mm, F.Cu at (277.9, 369.4)
- added B13: MK4096, Package_DIP:DIP-16_W7.62mm, F.Cu at (288.7, 369.4)
- added B14: MK4096, Package_DIP:DIP-16_W7.62mm, F.Cu at (245.6, 391.3)
- added B15: MK4096, Package_DIP:DIP-16_W7.62mm, F.Cu at (256.4, 391.3)
- added B16: MK4096, Package_DIP:DIP-16_W7.62mm, F.Cu at (267.1, 391.3)
- added B17: MK4096, Package_DIP:DIP-16_W7.62mm, F.Cu at (277.9, 391.3)
- added B18: MK4096, Package_DIP:DIP-16_W7.62mm, F.Cu at (288.7, 391.3)
- added B2: 7410, Package_DIP:DIP-14_W7.62mm, F.Cu at (409.1, 349.1)
- added B3: 74123, Package_DIP:DIP-16_W7.62mm, F.Cu at (56.9, 234.0)
- added B9: 74154, Package_DIP:DIP-24_W15.24mm, F.Cu at (225.3, 377.3)
- added C1: 7404, Package_DIP:DIP-14_W7.62mm, F.Cu at (419.9, 349.1)
- added C10: 7402, Package_DIP:DIP-14_W7.62mm, F.Cu at (463.0, 349.1)
- added C12: 7408, Package_DIP:DIP-14_W7.62mm, F.Cu at (481.9, 203.8)
- added C13: 74175, Package_DIP:DIP-16_W7.62mm, F.Cu at (492.7, 179.9)
- added C14: 74157, Package_DIP:DIP-16_W7.62mm, F.Cu at (503.4, 179.9)
- added C15: 7400, Package_DIP:DIP-14_W7.62mm, F.Cu at (500.4, 275.6)
- added C4: 74157, Package_DIP:DIP-16_W7.62mm, F.Cu at (481.9, 179.9)
- added C5: 7427, Package_DIP:DIP-14_W7.62mm, F.Cu at (430.6, 349.1)
- added C6: 7410, Package_DIP:DIP-14_W7.62mm, F.Cu at (441.4, 349.1)
- added C7: 74174, Package_DIP:DIP-16_W7.62mm, F.Cu at (31.6, 203.0)
- added C8: 7450, Package_DIP:DIP-14_W7.62mm, F.Cu at (58.7, 185.6)
- added C9: 7432, Package_DIP:DIP-14_W7.62mm, F.Cu at (452.2, 349.1)
- added CAP1: 0.01u, Capacitor_THT:C_Disc_D16.0mm_W5.0mm_P7.50mm, F.Cu at (95.0, 54.8)
- added CAP10: 0.01u, Capacitor_THT:C_Disc_D16.0mm_W5.0mm_P7.50mm, F.Cu at (114.6, 67.9)
- added CAP11: 0.01u, Capacitor_THT:C_Disc_D16.0mm_W5.0mm_P7.50mm, F.Cu at (114.6, 74.4)
- added CAP2: 0.01u, Capacitor_THT:C_Disc_D16.0mm_W5.0mm_P7.50mm, F.Cu at (95.0, 61.3)
- added CAP3: 0.01u, Capacitor_THT:C_Disc_D16.0mm_W5.0mm_P7.50mm, F.Cu at (95.0, 67.9)
- added CAP4: 0.01u, Capacitor_THT:C_Disc_D16.0mm_W5.0mm_P7.50mm, F.Cu at (95.0, 74.4)
- added CAP8: 0.01u, Capacitor_THT:C_Disc_D16.0mm_W5.0mm_P7.50mm, F.Cu at (114.6, 53.5)
- added CAP9: 0.01u, Capacitor_THT:C_Disc_D16.0mm_W5.0mm_P7.50mm, F.Cu at (114.6, 61.3)
- added D1: 74166, Package_DIP:DIP-16_W7.62mm, F.Cu at (514.2, 179.9)
- added D10: 7400, Package_DIP:DIP-14_W7.62mm, F.Cu at (511.1, 275.6)
- added D11: 74161, Package_DIP:DIP-16_W7.62mm, F.Cu at (568.1, 179.9)
- added D12: 7404, Package_DIP:DIP-14_W7.62mm, F.Cu at (473.8, 349.1)
- added D15: 74161, Package_DIP:DIP-16_W7.62mm, F.Cu at (578.9, 179.9)
- added D6: 74160, Package_DIP:DIP-16_W7.62mm, F.Cu at (525.0, 179.9)
- added D7: 74161, Package_DIP:DIP-16_W7.62mm, F.Cu at (535.8, 179.9)
- added D8: 74161, Package_DIP:DIP-16_W7.62mm, F.Cu at (546.6, 179.9)
- added D9: 74161, Package_DIP:DIP-16_W7.62mm, F.Cu at (557.3, 179.9)
- added R1: 1.5k, Resistor_THT:R_Axial_DIN0207_L6.3mm_D2.5mm_P10.16mm_Horizontal, F.Cu at (366.6, 347.0)
- added R10: 10k, Resistor_THT:R_Axial_DIN0207_L6.3mm_D2.5mm_P10.16mm_Horizontal, F.Cu at (366.6, 351.1)
- added R11: 10k, Resistor_THT:R_Axial_DIN0207_L6.3mm_D2.5mm_P10.16mm_Horizontal, F.Cu at (366.6, 355.1)
- added R13: 390, Resistor_THT:R_Axial_DIN0207_L6.3mm_D2.5mm_P10.16mm_Horizontal, F.Cu at (366.6, 359.2)
- added R14: 390, Resistor_THT:R_Axial_DIN0207_L6.3mm_D2.5mm_P10.16mm_Horizontal, F.Cu at (366.6, 363.2)
- added R15: 330, Resistor_THT:R_Axial_DIN0207_L6.3mm_D2.5mm_P10.16mm_Horizontal, F.Cu at (366.6, 367.3)
- added R2: 3k, Resistor_THT:R_Axial_DIN0207_L6.3mm_D2.5mm_P10.16mm_Horizontal, F.Cu at (330.1, 347.5)
- added R24: 3k, Resistor_THT:R_Axial_DIN0207_L6.3mm_D2.5mm_P10.16mm_Horizontal, F.Cu at (345.4, 347.5)
- added R25: 3k, Resistor_THT:R_Axial_DIN0207_L6.3mm_D2.5mm_P10.16mm_Horizontal, F.Cu at (345.4, 351.6)
- added R26: 3k, Resistor_THT:R_Axial_DIN0207_L6.3mm_D2.5mm_P10.16mm_Horizontal, F.Cu at (345.4, 355.6)
- added R27: 3k, Resistor_THT:R_Axial_DIN0207_L6.3mm_D2.5mm_P10.16mm_Horizontal, F.Cu at (345.4, 359.7)
- added R28: 27k, Resistor_THT:R_Axial_DIN0207_L6.3mm_D2.5mm_P10.16mm_Horizontal, F.Cu at (381.9, 347.0)
- added R29: 10k, Resistor_THT:R_Axial_DIN0207_L6.3mm_D2.5mm_P10.16mm_Horizontal, F.Cu at (381.9, 351.1)
- added R3: 3k, Resistor_THT:R_Axial_DIN0207_L6.3mm_D2.5mm_P10.16mm_Horizontal, F.Cu at (330.1, 351.6)
- added R31: 7.5k, Resistor_THT:R_Axial_DIN0207_L6.3mm_D2.5mm_P10.16mm_Horizontal, F.Cu at (366.6, 371.3)
- added R32: 7.5k, Resistor_THT:R_Axial_DIN0207_L6.3mm_D2.5mm_P10.16mm_Horizontal, F.Cu at (366.6, 375.4)
- added R33: 7.5k, Resistor_THT:R_Axial_DIN0207_L6.3mm_D2.5mm_P10.16mm_Horizontal, F.Cu at (366.6, 379.4)
- added R34: 7.5k, Resistor_THT:R_Axial_DIN0207_L6.3mm_D2.5mm_P10.16mm_Horizontal, F.Cu at (366.6, 383.5)
- added R35: 7.5k, Resistor_THT:R_Axial_DIN0207_L6.3mm_D2.5mm_P10.16mm_Horizontal, F.Cu at (366.6, 387.5)
- added R36: 7.5k, Resistor_THT:R_Axial_DIN0207_L6.3mm_D2.5mm_P10.16mm_Horizontal, F.Cu at (366.6, 391.6)
- added R4: 3k, Resistor_THT:R_Axial_DIN0207_L6.3mm_D2.5mm_P10.16mm_Horizontal, F.Cu at (330.1, 355.6)
- added R5: 3k, Resistor_THT:R_Axial_DIN0207_L6.3mm_D2.5mm_P10.16mm_Horizontal, F.Cu at (330.1, 359.7)
- added R6: 3k, Resistor_THT:R_Axial_DIN0207_L6.3mm_D2.5mm_P10.16mm_Horizontal, F.Cu at (330.1, 363.7)
- added R7: 3k, Resistor_THT:R_Axial_DIN0207_L6.3mm_D2.5mm_P10.16mm_Horizontal, F.Cu at (330.1, 367.8)
- added R8: 3k, Resistor_THT:R_Axial_DIN0207_L6.3mm_D2.5mm_P10.16mm_Horizontal, F.Cu at (330.1, 371.8)
- added R9: 3k, Resistor_THT:R_Axial_DIN0207_L6.3mm_D2.5mm_P10.16mm_Horizontal, F.Cu at (330.1, 375.9)
- moved A7 58.8 mm to (232.7, 344.3)
- moved A4 56.8 mm to (171.7, 342.3)
