File: mainboard/apple1.kicad_pcb (KiCad board)
At the start: 2 copper layers, 393.7 x 228.6 mm, 116 parts, among them J1 Conn_01x06, J2 Conn_01x04

Commit message: Progress 20260526
Parts:
- added B4: KEYBOARD, Package_DIP:DIP-16_W7.62mm, F.Cu at (150.8, 248.7)
- added CR1: 1N914, Diode_THT:D_DO-35_SOD27_P10.16mm_Horizontal, F.Cu at (364.2, 163.6)
- added CR2: 1N914, Diode_THT:D_DO-35_SOD27_P10.16mm_Horizontal, F.Cu at (364.2, 166.1)
- added CR3: 1N914, Diode_THT:D_DO-35_SOD27_P10.16mm_Horizontal, F.Cu at (364.2, 161.1)
- added CR4: 1N914, Diode_THT:D_DO-35_SOD27_P10.16mm_Horizontal, F.Cu at (260.1, 196.0)
- added DI5: 1N4001, Diode_THT:D_DO-41_SOD81_P10.16mm_Horizontal, F.Cu at (476.4, 151.2)
- added DI6: 1N4001, Diode_THT:D_DO-41_SOD81_P10.16mm_Horizontal, F.Cu at (476.4, 155.5)
- added DI7: 1N4001, Diode_THT:D_DO-41_SOD81_P10.16mm_Horizontal, F.Cu at (476.4, 159.8)
- added DI8: 1N4001, Diode_THT:D_DO-41_SOD81_P10.16mm_Horizontal, F.Cu at (476.4, 164.0)
- added J3: EDAC 305-044-520-201, mainboard:307044520201, F.Cu at (514.5, 286.9)
- moved CAP34 38.1 mm to (401.5, 77.5), turned to 90 degrees
Routing:
- net (no net): track 2615.9 -> 3361.6 mm
- net Net-(J6-~): track 431.1 -> 0.00 mm, vias 5 -> 0
- net Net-(J7-~): track 381.6 -> 0.00 mm, vias 3 -> 0
- net unconnected-(B4-Pin_13-Pad13): vias 0 -> 1
- net Net-(A10A-~-Pad1): vias 6 -> 7
- net GND: vias 138 -> 141
- net +5V: vias 90 -> 93
