File: mainboard/apple1.kicad_pcb (KiCad board)
At the start: 2 copper layers, 393.7 x 228.6 mm, 126 parts, among them J1 Conn_01x06, J2 Conn_01x04, J3 EDAC 305-044-520-201

Commit message: Additional  work on mainboard
Parts:
- A1, A10, A11, A12, A13, A14, A15, A16, A17, A18, A2, A9, B11, B12, B13, B14, B15, B16, B17, B18, B3, B4, C13, C14, C3, C4, C7, D1, D11, D15, D6, D7, D8, D9: footprint Package_DIP:DIP-16_W7.62mm -> mainboard:apple-1_DIP-16_W7.62mm
- B1, B2, C1, C10, C12, C15, C5, C6, C8, C9, D10, D12: footprint Package_DIP:DIP-14_W7.62mm -> mainboard:apple-1_DIP-14_W7.62mm
- B5, B6, B7, B8: value 74157_257 -> 74S257; footprint Package_DIP:DIP-16_W7.62mm -> mainboard:apple-1_DIP-16_W7.62mm
- C11A1, C11B1, D13, D14A1, D14B1, D4A1, D4B1, D5A1, D5B1: footprint Package_DIP:DIP-8_W7.62mm -> mainboard:apple-1_DIP-8_W7.62mm
- J2: footprint Connector_JST:JST_VH_B4P-VH_1x04_P3.96mm_Vertical -> mainboard:apple-1_JST_VH_B4P-VH_1x04_P3.96mm_Vertical
- R1, R10, R11, R13, R14, R15, R16, R17, R18, R19, R2, R20, R21, R22, R23, R24, R25, R26, R27, R28, R29, R3, R31, R32, R33, R34, R35, R36, R4, R5, R6, R7, R8, R9: footprint Resistor_THT:R_Axial_DIN0207_L6.3mm_D2.5mm_P10.16mm_Horizontal -> mainboard:apple-1_R_Axial_DIN0207_L6.3mm_D2.5mm_P10.16mm_Horizontal
- moved CAP1 622.4 mm to (654.2, -202.7)
- moved CAP10 622.4 mm to (667.3, -222.3)
- moved CAP11 622.4 mm to (673.9, -222.3)
- moved CAP2 622.4 mm to (660.8, -202.7)
- moved CAP3 622.4 mm to (667.3, -202.7)
- moved CAP4 622.4 mm to (673.9, -202.7)
- moved CAP8 622.4 mm to (653.0, -222.3)
- moved CAP9 622.4 mm to (660.8, -222.3)
- moved CAP35 479.5 mm to (713.0, -259.4)
- moved CAP36 479.5 mm to (713.0, -251.4)
- moved CAP37 479.5 mm to (713.0, -243.3)
- moved CAP34 465.9 mm to (748.5, -233.4)
- moved DI5 372.9 mm to (675.4, -164.2)
- moved DI6 372.9 mm to (675.4, -159.9)
- moved DI7 372.9 mm to (675.4, -155.7)
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Other:
- board text added: "(6800 ONLY)"
