File: mainboard/mainboard.kicad_pcb (KiCad board)
At the start: 2 copper layers, 393.7 x 228.6 mm, 131 parts, among them J1 Conn_01x06, J2 Conn_01x04, J3 EDAC 305-044-520-201

Commit message: removing overlapping footprint geometry
Routing:
- net +5V: track 10888.5 -> 10887.4 mm, vias 90 -> 46
- net GND: track 53581.7 -> 53581.1 mm, vias 137 -> 91
- net Net-(A13-DOUT): track 144.3 -> 143.7 mm, vias 4 -> 1
- net /Processor Section/A7_1: track 983.7 -> 983.0 mm, vias 23 -> 4
- net ~{RDA}: vias 3 -> 2
- net unconnected-(D1-Clr-Pad9): vias 1 -> 0
- net unconnected-(C7-~{Mr}-Pad1): vias 1 -> 0
- net unconnected-(C14-Zb-Pad7): vias 1 -> 0
- net unconnected-(C14-I1b-Pad6): vias 1 -> 0
- net unconnected-(C14-I0b-Pad5): vias 1 -> 0
- net unconnected-(C13-~{Mr}-Pad1): vias 1 -> 0
- net unconnected-(C13-Q3-Pad15): vias 1 -> 0
- net unconnected-(C13-Q2-Pad10): vias 1 -> 0
- net unconnected-(C13-Q1-Pad7): vias 1 -> 0
- net unconnected-(C13-Q0-Pad2): vias 1 -> 0
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