File: mainboard/mainboard.kicad_pcb (KiCad board)
At the start: 2 copper layers, 393.7 x 228.6 mm, 172 parts, among them J1 Conn_01x06, J12 Y, J13 Conn_01x16, J2 Conn_01x04, J3 EDAC 305-044-520-201, J4 W, J5 X, J6 S, J7 R, J8 T, J9 Z, Q1 Q_NPN_EBC, Q2 Q_PNP_EBC, Q3 Q_NPN_EBC, Q4 Q_PNP_EBC, Q5 MPS3704, Y1 14.31818 MHz

Commit message: board is now complete, cleanup work can begin
Parts:
- moved C29 7.62 mm to (378.4, 148.0), turned to -90 degrees
- moved C25 7.62 mm to (234.9, 294.6), turned to -90 degrees
- moved C28 7.62 mm to (234.9, 194.3), turned to -90 degrees
- moved C30 7.62 mm to (234.9, 147.3), turned to -90 degrees
- moved C26 7.62 mm to (234.9, 243.2), turned to -90 degrees
- moved C27 7.62 mm to (378.5, 195.6), turned to -90 degrees
Connections:
- B4 pad 11: /Processor Section/-12V -> -12V
- C25 pad 1: +5V -> GND
- C25 pad 2: GND -> +5V
- C26 pad 1: +5V -> GND
- C26 pad 2: GND -> +5V
- C27 pad 1: +5V -> GND
- C27 pad 2: GND -> +5V
- C28 pad 1: +5V -> GND
- C28 pad 2: GND -> +5V
- C29 pad 1: +5V -> GND
- C29 pad 2: GND -> +5V
- C30 pad 1: +5V -> GND
- C30 pad 2: GND -> +5V
- J12 pad 22: (no net) -> Net-(A1-~{CS1})
- J4 pad 20: (no net) -> Net-(A11-~{CS})
- J5 pad 21: (no net) -> Net-(B11-~{CS})
- J6 pad 18: (no net) -> Net-(J6-~)
- J8 pad 19: (no net) -> Net-(J8-~)
- J9 pad 23: (no net) -> Net-(A4-~{CS2})
- R29 pad 1: Net-(B3B-Cext) -> Net-(B3B-RCext)
Routing:
- net GND: track 2543.1 -> 3263.4 mm
- net Net-(A18-DOUT): track 237.7 -> 233.4 mm
Other:
- board text added: "BOARD TEXT PROOF AREA:"
