File: mainboard/processor.kicad_sch (KiCad schematic)
At the start: 83 parts, among them J10 6502, J11 6502, J12 Y, J13 Conn_01x16, J14 NO DMA, J3 EdgeConnector, J4 W, J5 X, J6 S, J7 R, J8 T, J9 Z, Q1 Q_NPN_EBC, Q2 Q_PNP_EBC, Q3 Q_NPN_EBC, Q4 Q_PNP_EBC

Commit message: Further work on the schematics/file organization
Parts:
- A1, A11, A12, A13, A14, A15, A16, A17, A18, A2, B11, B12, B13, B14, B15, B16, B17, B18, B3: footprint ~ -> Package_DIP:DIP-16_W7.62mm
- A4: Comment (none) -> Alt: 6520
- A7: Comment (none) -> OEM: Mostek
- B1, B2, C1, C15, D10: footprint ~ -> Package_DIP:DIP-14_W7.62mm
- B9: footprint ~ -> Package_DIP:DIP-24_W15.24mm
- CAP10, CAP11, CAP8, CAP9: footprint ~ -> Capacitor_THT:C_Disc_D16.0mm_W5.0mm_P7.50mm; Comment (none) -> ALT: BC2361-ND
- CAP12, CAP13, CAP14, CAP15, CAP16, CAP17, CAP18, CAP19, CAP20, CAP21, CAP22, CAP23, CAP24: Comment (none) -> .3 LEAD SPACING
- J3: Comment (none) -> .2X.140 SPACING
- R24, R25, R26, R27, R28, R29: footprint ~ -> Resistor_THT:R_Axial_DIN0207_L6.3mm_D2.5mm_P10.16mm_Horizontal

Commit message: Additional  work on mainboard
Parts:
- A10, A9, B5, B6, B7, B8: footprint ~ -> Package_DIP:DIP-16_W7.62mm
- B4, CAP12, CAP13, CAP14, CAP15, CAP16, CAP17, CAP18, CAP19, CAP20, CAP21, CAP22, CAP23, CAP24, J10, J11, J12, J13, J14, J4, J5, J6, J7, J8, J9, JP1, JP2, Q1, Q2, Q3, Q4: footprint ~ -> (none)
- J3: value EdgeConnector -> EDAC 305-044-520-201; footprint ~ -> mainboard:307044520201; Comment .2X.140 SPACING -> (none)
- R16, R17, R18, R19: value 1k -> 1K; footprint ~ -> Resistor_THT:R_Axial_DIN0207_L6.3mm_D2.5mm_P10.16mm_Horizontal
- R20, R21, R22, R23: footprint ~ -> Resistor_THT:R_Axial_DIN0207_L6.3mm_D2.5mm_P10.16mm_Horizontal
- R24, R25, R26, R27: value 3k -> 3K
- R28: value 27k -> 27K
- R29: value 10k -> 10K

Commit message: Progress 20260526
Parts:
- B4: footprint (none) -> Package_DIP:DIP-16_W7.62mm
Changed lines of the file:
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@@
 			)
 		)
-		(property "Footprint" ""
+		(property "Footprint" "Package_DIP:DIP-16_W7.62mm"
 			(at 167.64 218.44 0)
 			(hide yes)

Commit message: Additional  work on mainboard
Parts:
- A1, A10, A11, A12, A13, A14, A15, A16, A17, A18, A2, A9, B11, B12, B13, B14, B15, B16, B17, B18, B3, B4: footprint Package_DIP:DIP-16_W7.62mm -> mainboard:apple-1_DIP-16_W7.62mm
- B1, B2, C1, C15, D10: footprint Package_DIP:DIP-14_W7.62mm -> mainboard:apple-1_DIP-14_W7.62mm
- B5, B6, B7, B8: value 74157_257 -> 74S257; footprint Package_DIP:DIP-16_W7.62mm -> mainboard:apple-1_DIP-16_W7.62mm
- R16, R17, R18, R19, R20, R21, R22, R23, R24, R25, R26, R27, R28, R29: footprint Resistor_THT:R_Axial_DIN0207_L6.3mm_D2.5mm_P10.16mm_Horizontal -> mainboard:apple-1_R_Axial_DIN0207_L6.3mm_D2.5mm_P10.16mm_Horizontal

Commit message: 20260605
Parts:
- CAP10, CAP11, CAP8, CAP9: footprint Capacitor_THT:C_Disc_D16.0mm_W5.0mm_P7.50mm -> mainboard:apple-1_C_Disc_D16.0mm_W5.0mm_P7.50mm
