File: mainboard/processor.kicad_sch (KiCad schematic)
At the start: 83 parts, among them J10 6502, J11 6502, J12 Y, J13 Conn_01x16, J14 NO DMA, J3 EDAC 305-044-520-201, J4 W, J5 X, J6 S, J7 R, J8 T, J9 Z, Q1 Q_NPN_EBC, Q2 Q_PNP_EBC, Q3 Q_NPN_EBC, Q4 Q_PNP_EBC

Commit message: Additional footprint and filled zone work on mainboard.
Parts:
- A4, A7: footprint Package_DIP:DIP-40_W15.24mm -> mainboard:apple-1_DIP-40_W15.24mm
- B9: footprint Package_DIP:DIP-24_W15.24mm -> mainboard:apple-1_DIP-24_18.0mmx34.29mm_W15.24mm
Changed lines of the file:
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@@
 			)
 		)
-		(property "Footprint" "Package_DIP:DIP-40_W15.24mm"
+		(property "Footprint" "mainboard:apple-1_DIP-40_W15.24mm"
 			(at 335.28 266.7 0)
 			(hide yes)
@@
 			)
 		)
-		(property "Footprint" "Package_DIP:DIP-24_W15.24mm"
+		(property "Footprint" "mainboard:apple-1_DIP-24_18.0mmx34.29mm_W15.24mm"
 			(at 454.66 342.9 0)
 			(hide yes)
@@
 			)
 		)
-		(property "Footprint" "Package_DIP:DIP-40_W15.24mm"
+		(property "Footprint" "mainboard:apple-1_DIP-40_W15.24mm"
 			(at 132.08 271.78 0)
 			(hide yes)

Commit message: more work on mainboard
Parts:
- CAP10: value 0.01u -> .01; footprint mainboard:apple-1_C_Disc_D16.0mm_W5.0mm_P7.50mm -> mainboard:apple-1_C_Disc_D16.0mm_W5.0mm_P7.50mm (68000 section); PCBDisplay (none) -> C10
- CAP11: value 0.01u -> .01; footprint mainboard:apple-1_C_Disc_D16.0mm_W5.0mm_P7.50mm -> mainboard:apple-1_C_Disc_D16.0mm_W5.0mm_P7.50mm (68000 section); PCBDisplay (none) -> C11
- CAP12: value 1u -> 1.0; footprint (none) -> mainboard:apple-1_C_Disc_D16.0mm_W5.0mm_P7.50mm (68000 section); PCBDisplay (none) -> C12
- CAP13: value 1u -> 1.0; footprint (none) -> mainboard:apple-1_C_Disc_D16.0mm_W5.0mm_P7.50mm (68000 section); PCBDisplay (none) -> C13
- CAP14, CAP15, CAP16, CAP17, CAP18, CAP21, CAP22, CAP23, CAP24: footprint (none) -> mainboard:apple-1_C_Disc_D16.0mm_W5.0mm_P7.50mm
- CAP19: value 47p -> 47PF; footprint (none) -> mainboard:apple-1_C_Disc_D16.0mm_W5.0mm_P7.50mm
- CAP20: value 0.001u -> .001; footprint (none) -> mainboard:apple-1_C_Disc_D16.0mm_W5.0mm_P7.50mm
- CAP8: value 0.01u -> .01; footprint mainboard:apple-1_C_Disc_D16.0mm_W5.0mm_P7.50mm -> mainboard:apple-1_C_Disc_D16.0mm_W5.0mm_P7.50mm (68000 section); PCBDisplay (none) -> C8
- CAP9: value 0.01u -> .01; footprint mainboard:apple-1_C_Disc_D16.0mm_W5.0mm_P7.50mm -> mainboard:apple-1_C_Disc_D16.0mm_W5.0mm_P7.50mm (68000 section); PCBDisplay (none) -> C9
- J13: footprint (none) -> mainboard:J13
Connections:
- net at B3.6 (Cext), R29.1: now also CAP20.2; no longer CAP20.1
- net at B3.7 (RCext): now also CAP20.1; no longer CAP20.2

Commit message: additional footprint work
Parts:
- C10: renamed from CAP10; PCBDisplay C10 -> (none)
- C11: renamed from CAP11; PCBDisplay C11 -> (none)
- C12: renamed from CAP12; Comment .3 LEAD SPACING -> (none); PCBDisplay C12 -> (none)
- C13: renamed from CAP13; Comment .3 LEAD SPACING -> (none); PCBDisplay C13 -> (none)
- C14: renamed from CAP14; Comment .3 LEAD SPACING -> (none)
- C15: renamed from CAP15; Comment .3 LEAD SPACING -> (none)
- C16: renamed from CAP16; Comment .3 LEAD SPACING -> (none)
- C17: renamed from CAP17; Comment .3 LEAD SPACING -> (none)
- C18: renamed from CAP18; Comment .3 LEAD SPACING -> (none)
- C19: renamed from CAP19; Comment .3 LEAD SPACING -> (none)
- C20: renamed from CAP20; Comment .3 LEAD SPACING -> (none)
- C21: renamed from CAP21; Comment .3 LEAD SPACING -> (none)
- C22: renamed from CAP22; Comment .3 LEAD SPACING -> (none)
- C23: renamed from CAP23; Comment .3 LEAD SPACING -> (none)
- C24: renamed from CAP24; Comment .3 LEAD SPACING -> (none)
- C8: renamed from CAP8; PCBDisplay C8 -> (none)
- C9: renamed from CAP9; PCBDisplay C9 -> (none)
- J12: footprint (none) -> mainboard:YJumper
- J4: footprint (none) -> mainboard:WJumper
- J5: footprint (none) -> mainboard:XJumper
- J6: footprint (none) -> mainboard:SJumper
- J7: footprint (none) -> mainboard:RJumper
- J8: footprint (none) -> mainboard:TJumper
- J9: footprint (none) -> mainboard:ZJumper
- Q1, Q2, Q3, Q4: footprint (none) -> mainboard:apple-1_TO-92_HandSolder
- renumbered C1 to C_IC1, C15 to C_IC15
