File: mainboard/terminal.kicad_sch (KiCad schematic)
At the start: 67 parts, among them J2 Conn_01x04, Q5 MPS3704, Y1 14.31818 MHz

Commit message: Further work on the schematics/file organization
Parts:
- B2, C10, C12, C15, C5, C6, C8, C9, D10, D12: footprint ~ -> Package_DIP:DIP-14_W7.62mm
- C13, C14, C4, C7, D1, D11, D15, D6, D7, D8, D9: footprint ~ -> Package_DIP:DIP-16_W7.62mm
- CAP1, CAP2, CAP3, CAP4: footprint ~ -> Capacitor_THT:C_Disc_D16.0mm_W5.0mm_P7.50mm; Comment (none) -> ALT: BC2361-ND
- CAP7: Comment (none) -> .3 LEAD SPACING
- R1, R2: footprint (none) -> Resistor_THT:R_Axial_DIN0207_L6.3mm_D2.5mm_P10.16mm_Horizontal
- R10, R11, R13, R14, R15, R3, R31, R32, R33, R34, R35, R36, R4, R5, R6, R7, R8, R9: footprint ~ -> Resistor_THT:R_Axial_DIN0207_L6.3mm_D2.5mm_P10.16mm_Horizontal

Commit message: Additional  work on mainboard
Parts:
- C11A1, C11B1, D13, D14A1, D14B1, D4A1, D4B1, D5A1, D5B1: footprint ~ -> Package_DIP:DIP-8_W7.62mm
- C3: footprint ~ -> Package_DIP:DIP-16_W7.62mm
- CAP5, CAP6, CAP7, CR1, CR2, CR3, CR4, Q5, R12, Y1: footprint ~ -> (none)
- D2: footprint ~ -> Package_DIP:DIP-24_18.0mmx34.29mm_W15.24mm
- J2: footprint ~ -> Connector_JST:JST_VH_B4P-VH_1x04_P3.96mm_Vertical
- R1: value 1.5k -> 1.5K
- R10, R11: value 10k -> 10K
- R2, R3, R4, R5, R6, R7, R8, R9: value 3k -> 3K
- R31, R32, R33, R34, R35, R36: value 7.5k -> 7.5K

Commit message: Progress 20260526
Parts:
- CR1, CR2, CR3, CR4: footprint (none) -> Diode_THT:D_DO-35_SOD27_P10.16mm_Horizontal
Changed lines of the file:
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@@
 			)
 		)
-		(property "Footprint" ""
+		(property "Footprint" "Diode_THT:D_DO-35_SOD27_P10.16mm_Horizontal"
 			(at 241.3 243.205 0)
 			(hide yes)
@@
 			)
 		)
-		(property "Footprint" ""
+		(property "Footprint" "Diode_THT:D_DO-35_SOD27_P10.16mm_Horizontal"
 			(at 241.3 245.745 0)
 			(hide yes)
@@
 			)
 		)
-		(property "Footprint" ""
+		(property "Footprint" "Diode_THT:D_DO-35_SOD27_P10.16mm_Horizontal"
 			(at 241.3 248.285 0)
 			(hide yes)
@@
 			)
 		)
-		(property "Footprint" ""
+		(property "Footprint" "Diode_THT:D_DO-35_SOD27_P10.16mm_Horizontal"
 			(at 495.935 210.82 0)
 			(hide yes)

Commit message: Additional  work on mainboard
Parts:
- B2, C10, C12, C15, C5, C6, C8, C9, D10, D12: footprint Package_DIP:DIP-14_W7.62mm -> mainboard:apple-1_DIP-14_W7.62mm
- C11A1, C11B1, D13, D14A1, D14B1, D4A1, D4B1, D5A1, D5B1: footprint Package_DIP:DIP-8_W7.62mm -> mainboard:apple-1_DIP-8_W7.62mm
- C13, C14, C3, C4, C7, D1, D11, D15, D6, D7, D8, D9: footprint Package_DIP:DIP-16_W7.62mm -> mainboard:apple-1_DIP-16_W7.62mm
- J2: footprint Connector_JST:JST_VH_B4P-VH_1x04_P3.96mm_Vertical -> mainboard:apple-1_JST_VH_B4P-VH_1x04_P3.96mm_Vertical
- R1, R10, R11, R13, R14, R15, R2, R3, R31, R32, R33, R34, R35, R36, R4, R5, R6, R7, R8, R9: footprint Resistor_THT:R_Axial_DIN0207_L6.3mm_D2.5mm_P10.16mm_Horizontal -> mainboard:apple-1_R_Axial_DIN0207_L6.3mm_D2.5mm_P10.16mm_Horizontal

Commit message: large renaming, tidying up files, old libraries
Parts:
- D13: value NE555 -> 555
- Y1: footprint (none) -> Crystal:Resonator-2Pin_W10.0mm_H5.0mm
Changed lines of the file:
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@@
 			)
 		)
-		(property "Footprint" ""
+		(property "Footprint" "Crystal:Resonator-2Pin_W10.0mm_H5.0mm"
 			(at 72.39 365.76 0)
 			(hide yes)
@@
 			)
 		)
-		(property "Value" "NE555"
+		(property "Value" "555"
 			(at 231.14 335.915 0)
 			(show_name no)

Commit message: 20260605
Parts:
- CAP1, CAP2, CAP3, CAP4: footprint Capacitor_THT:C_Disc_D16.0mm_W5.0mm_P7.50mm -> mainboard:apple-1_C_Disc_D16.0mm_W5.0mm_P7.50mm
