File: mainboard/terminal.kicad_sch (KiCad schematic)
At the start: 67 parts, among them J2 Conn_01x04, Q5 MPS3704, Y1 14.31818 MHz

Commit message: Additional footprint and filled zone work on mainboard.
Parts:
- CR1, CR2, CR3, CR4: footprint Diode_THT:D_DO-35_SOD27_P10.16mm_Horizontal -> mainboard:apple-1_D_DO-35_SOD27_P10.16mm_Horizontal
- D2: footprint Package_DIP:DIP-24_18.0mmx34.29mm_W15.24mm -> mainboard:apple-1_DIP-24_18.0mmx34.29mm_W15.24mm
Changed lines of the file:
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@@
 			)
 		)
-		(property "Footprint" "Diode_THT:D_DO-35_SOD27_P10.16mm_Horizontal"
+		(property "Footprint" "mainboard:apple-1_D_DO-35_SOD27_P10.16mm_Horizontal"
 			(at 241.3 243.205 0)
 			(hide yes)
@@
 			)
 		)
-		(property "Footprint" "Diode_THT:D_DO-35_SOD27_P10.16mm_Horizontal"
+		(property "Footprint" "mainboard:apple-1_D_DO-35_SOD27_P10.16mm_Horizontal"
 			(at 241.3 245.745 0)
 			(hide yes)
@@
 			)
 		)
-		(property "Footprint" "Diode_THT:D_DO-35_SOD27_P10.16mm_Horizontal"
+		(property "Footprint" "mainboard:apple-1_D_DO-35_SOD27_P10.16mm_Horizontal"
 			(at 241.3 248.285 0)
 			(hide yes)
@@
 			)
 		)
-		(property "Footprint" "Diode_THT:D_DO-35_SOD27_P10.16mm_Horizontal"
+		(property "Footprint" "mainboard:apple-1_D_DO-35_SOD27_P10.16mm_Horizontal"
 			(at 495.935 210.82 0)
 			(hide yes)
@@
 			)
 		)
-		(property "Footprint" "Package_DIP:DIP-24_18.0mmx34.29mm_W15.24mm"
+		(property "Footprint" "mainboard:apple-1_DIP-24_18.0mmx34.29mm_W15.24mm"
 			(at 203.2 168.91 0)
 			(hide yes)

Commit message: more work on mainboard
Parts:
- CAP1, CAP2, CAP3, CAP4: value 0.01u -> .01
- CAP5, CAP6: value 1u -> 1.0; footprint (none) -> mainboard:apple-1_C_Disc_D16.0mm_W5.0mm_P7.50mm
