File: mainboard/power_supply.kicad_sch (KiCad schematic)
At the start: 35 parts, among them J1 Conn_01x06

Commit message: Additional footprint and filled zone work on mainboard.
Parts:
- CAP32: value 2400u -> 2400UF; footprint mainboard:apple-1_CP_Axial_L55.0mm_D26.0mm_P55.88mm_Horizontal -> mainboard:apple-1_CP_2400UF_25V_-+
- CAP33: value 2400u -> 2400UF
- DI1, DI2, DI3, DI4: value MR500 -> MR 500; footprint Diode_THT:D_5W_P10.16mm_Horizontal -> mainboard:apple-1_D_5W_P10.16mm_Horizontal
Changed lines of the file:
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@@
 			)
 		)
-		(property "Value" "MR500"
+		(property "Value" "MR 500"
 			(at 102.87 36.83 0)
 			(show_name no)
@@
 			)
 		)
-		(property "Footprint" "Diode_THT:D_5W_P10.16mm_Horizontal"
+		(property "Footprint" "mainboard:apple-1_D_5W_P10.16mm_Horizontal"
 			(at 97.79 38.1 0)
 			(hide yes)
@@
 			)
 		)
-		(property "Value" "MR500"
+		(property "Value" "MR 500"
 			(at 102.87 41.91 0)
 			(show_name no)
@@
 			)
 		)
-		(property "Footprint" "Diode_THT:D_5W_P10.16mm_Horizontal"
+		(property "Footprint" "mainboard:apple-1_D_5W_P10.16mm_Horizontal"
 			(at 97.79 43.18 0)
 			(hide yes)
@@
 			)
 		)
-		(property "Value" "MR500"
+		(property "Value" "MR 500"
 			(at 102.87 46.99 0)
 			(show_name no)
@@
 			)
 		)
-		(property "Footprint" "Diode_THT:D_5W_P10.16mm_Horizontal"
+		(property "Footprint" "mainboard:apple-1_D_5W_P10.16mm_Horizontal"
 			(at 97.79 48.26 0)
 			(hide yes)
@@
 			)
 		)
-		(property "Value" "2400u"
+		(property "Value" "2400UF"
 			(at 133.35 77.47 0)
 			(show_name no)
@@
 			)
 		)
-		(property "Footprint" "mainboard:apple-1_CP_Axial_L55.0mm_D26.0mm_P55.88mm_Horizontal"
+		(property "Footprint" "mainboard:apple-1_CP_2400UF_25V_-+"
 			(at 124.46 77.47 0)
 			(hide yes)
@@
 			)
 		)
-		(property "Value" "MR500"
+		(property "Value" "MR 500"
 			(at 102.87 52.07 0)
 			(show_name no)
@@
 			)
 		)
-		(property "Footprint" "Diode_THT:D_5W_P10.16mm_Horizontal"
+		(property "Footprint" "mainboard:apple-1_D_5W_P10.16mm_Horizontal"
 			(at 97.79 53.34 0)
 			(hide yes)
@@
 			)
 		)
-		(property "Value" "2400u"
+		(property "Value" "2400UF"
 			(at 127.635 98.425 0)
 			(show_name no)

Commit message: additional footprint refinement and mainboard update
Parts:
- CAP34, CAP35, CAP37: value 22u -> 22MF
- CAP36: value 22u -> 22MF; footprint Capacitor_THT:C_Axial_L12.0mm_D6.5mm_P20.00mm_Horizontal -> mainboard:apple-1_C_Axial_L12.0mm_D6.5mm_P20.00mm_Horizontal
- DI2, DI3: footprint mainboard:apple-1_D_5W_P10.16mm_Horizontal -> mainboard:apple-1_D_5W_P10.16mm_Horizontal_Mirrored
- DI5, DI8: footprint Diode_THT:D_DO-41_SOD81_P10.16mm_Horizontal -> mainboard:apple-1_D_5W_P10.16mm_Horizontal
- DI6, DI7: footprint Diode_THT:D_DO-41_SOD81_P10.16mm_Horizontal -> mainboard:apple-1_D_5W_P10.16mm_Horizontal_Mirrored
Changed lines of the file:
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@@
 			)
 		)
-		(property "Footprint" "mainboard:apple-1_D_5W_P10.16mm_Horizontal"
+		(property "Footprint" "mainboard:apple-1_D_5W_P10.16mm_Horizontal_Mirrored"
 			(at 97.79 43.18 0)
 			(hide yes)
@@
 			)
 		)
-		(property "Footprint" "mainboard:apple-1_D_5W_P10.16mm_Horizontal"
+		(property "Footprint" "mainboard:apple-1_D_5W_P10.16mm_Horizontal_Mirrored"
 			(at 97.79 48.26 0)
 			(hide yes)
@@
 			)
 		)
-		(property "Value" "22u"
+		(property "Value" "22MF"
 			(at 176.53 77.47 0)
 			(show_name no)
@@
 			)
 		)
-		(property "Footprint" "Capacitor_THT:C_Axial_L12.0mm_D6.5mm_P20.00mm_Horizontal"
+		(property "Footprint" "mainboard:apple-1_C_Axial_L12.0mm_D6.5mm_P20.00mm_Horizontal"
 			(at 170.18 77.47 0)
 			(hide yes)
@@
 			)
 		)
-		(property "Value" "22u"
+		(property "Value" "22MF"
 			(at 173.355 57.785 0)
 			(show_name no)
@@
 			)
 		)
-		(property "Value" "22u"
+		(property "Value" "22MF"
 			(at 176.53 36.83 0)
 			(show_name no)
@@
 			)
 		)
-		(property "Value" "22u"
+		(property "Value" "22MF"
 			(at 173.355 98.425 0)
 			(show_name no)
@@
 			)
 		)
-		(property "Footprint" "Diode_THT:D_DO-41_SOD81_P10.16mm_Horizontal"
+		(property "Footprint" "mainboard:apple-1_D_5W_P10.16mm_Horizontal"
 			(at 97.79 68.58 0)
 			(hide yes)
@@
 			)
 		)
-		(property "Footprint" "Diode_THT:D_DO-41_SOD81_P10.16mm_Horizontal"
+		(property "Footprint" "mainboard:apple-1_D_5W_P10.16mm_Horizontal_Mirrored"
 			(at 97.79 73.66 0)
 			(hide yes)
@@
 			)
 		)
-		(property "Footprint" "Diode_THT:D_DO-41_SOD81_P10.16mm_Horizontal"
+		(property "Footprint" "mainboard:apple-1_D_5W_P10.16mm_Horizontal_Mirrored"
 			(at 97.79 78.74 0)
 			(hide yes)
@@
 			)
 		)
-		(property "Footprint" "Diode_THT:D_DO-41_SOD81_P10.16mm_Horizontal"
+		(property "Footprint" "mainboard:apple-1_D_5W_P10.16mm_Horizontal"
 			(at 97.79 83.82 0)
 			(hide yes)
