File: mainboard/power_supply.kicad_sch (KiCad schematic)
At the start: 35 parts, among them J1 Conn_01x06

Commit message: more work on mainboard
Parts:
- CAP31: value 5300u -> 5300UF; footprint (none) -> mainboard:apple-1_CP_5300UF_15V_+-
- REG1: footprint Package_TO_SOT_THT:TO-220-3_Vertical -> mainboard:LM320 MP-5 (TO-220-3_Vertical_SpacedPins)
- REG3: footprint Package_TO_SOT_THT:TO-220-3_Vertical -> mainboard:LM320 MP-12 (TO-220-3_Vertical_SpacedPins)
- REG4: footprint Package_TO_SOT_THT:TO-220-3_Vertical -> mainboard:LM340-12 (TO-220-3_Vertical_SpacedPins)
Connections:
- net +12V: now also REG4.3 (OUT); no longer REG4.2 (OUT)
- net -12V: now also REG1.2 (IN), REG3.3 (OUT); no longer REG1.3 (IN), REG3.2 (OUT)
- net -12V_UNREG: now also REG3.2 (IN); no longer REG3.3 (IN)
- net -5V: now also REG1.3 (OUT); no longer REG1.2 (OUT)
- net GND: now also REG4.2 (GND); no longer REG4.3 (GND)

Commit message: additional footprint work
Parts:
- C31: renamed from CAP31; Comment .3 LEAD SPACING -> (none)
- C32: renamed from CAP32; Comment .3 LEAD SPACING -> (none)
- C33: renamed from CAP33; Comment .3 LEAD SPACING -> (none)
- C34: renamed from CAP34; footprint Capacitor_THT:C_Axial_L12.0mm_D6.5mm_P20.00mm_Horizontal -> mainboard:apple-1_C_Axial_22MF_25V_P1200mils_Horizontal; Comment .3 LEAD SPACING -> (none)
- C35: renamed from CAP35; footprint Capacitor_THT:C_Axial_L12.0mm_D6.5mm_P20.00mm_Horizontal -> mainboard:apple-1_C_Axial_22MF_25V_P1200mils_Horizontal; Comment .3 LEAD SPACING -> (none)
- C36: renamed from CAP36; Comment .3 LEAD SPACING -> (none)
- C37: renamed from CAP37; footprint Capacitor_THT:C_Axial_L12.0mm_D6.5mm_P20.00mm_Horizontal -> mainboard:apple-1_C_Axial_22MF_25V_P1200mils_Horizontal; Comment .3 LEAD SPACING -> (none)
- renumbered C1 to C_IC1, C10 to C_IC10, C12 to C_IC12, C15 to C_IC15, C5 to C_IC5, C6 to C_IC6, C8 to C_IC8, C9 to C_IC9

Commit message: mainboard work
Parts:
- C33: footprint mainboard:apple-1_CP_Axial_L55.0mm_D26.0mm_P55.88mm_Horizontal -> mainboard:apple-1_CP_2400UF_25V_-+
- C34, C37: footprint mainboard:apple-1_C_Axial_22MF_25V_P1200mils_Horizontal -> mainboard:apple-1_C_Axial_L12.0mm_D6.5mm_P20.00mm_Horizontal
- DI2, DI3, DI6, DI7: footprint mainboard:apple-1_D_5W_P10.16mm_Horizontal_Mirrored -> mainboard:apple-1_D_5W_P10.16mm_Horizontal
- J1: footprint Connector_JST:JST_VH_B6P-VH_1x06_P3.96mm_Vertical -> mainboard:apple-1_JST_VH_B6P-VH_1x06_P3.96mm_Vertical
Changed lines of the file:
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@@
 			)
 		)
-		(property "Footprint" "mainboard:apple-1_D_5W_P10.16mm_Horizontal_Mirrored"
+		(property "Footprint" "mainboard:apple-1_D_5W_P10.16mm_Horizontal"
 			(at 97.79 43.18 0)
 			(hide yes)
@@
 			)
 		)
-		(property "Footprint" "mainboard:apple-1_D_5W_P10.16mm_Horizontal_Mirrored"
+		(property "Footprint" "mainboard:apple-1_D_5W_P10.16mm_Horizontal"
 			(at 97.79 48.26 0)
 			(hide yes)
@@
 			)
 		)
-		(property "Footprint" "mainboard:apple-1_C_Axial_22MF_25V_P1200mils_Horizontal"
+		(property "Footprint" "mainboard:apple-1_C_Axial_L12.0mm_D6.5mm_P20.00mm_Horizontal"
 			(at 170.18 36.83 0)
 			(hide yes)
@@
 			)
 		)
-		(property "Footprint" "mainboard:apple-1_CP_Axial_L55.0mm_D26.0mm_P55.88mm_Horizontal"
+		(property "Footprint" "mainboard:apple-1_CP_2400UF_25V_-+"
 			(at 124.46 97.79 0)
 			(hide yes)
@@
 			)
 		)
-		(property "Footprint" "mainboard:apple-1_C_Axial_22MF_25V_P1200mils_Horizontal"
+		(property "Footprint" "mainboard:apple-1_C_Axial_L12.0mm_D6.5mm_P20.00mm_Horizontal"
 			(at 170.18 97.79 0)
 			(hide yes)
@@
 			)
 		)
-		(property "Footprint" "mainboard:apple-1_D_5W_P10.16mm_Horizontal_Mirrored"
+		(property "Footprint" "mainboard:apple-1_D_5W_P10.16mm_Horizontal"
 			(at 97.79 73.66 0)
 			(hide yes)
@@
 			)
 		)
-		(property "Footprint" "mainboard:apple-1_D_5W_P10.16mm_Horizontal_Mirrored"
+		(property "Footprint" "mainboard:apple-1_D_5W_P10.16mm_Horizontal"
 			(at 97.79 78.74 0)
 			(hide yes)
@@
 			)
 		)
-		(property "Footprint" "Connector_JST:JST_VH_B6P-VH_1x06_P3.96mm_Vertical"
+		(property "Footprint" "mainboard:apple-1_JST_VH_B6P-VH_1x06_P3.96mm_Vertical"
 			(at 58.42 55.88 0)
 			(hide yes)

Commit message: added kicad drawing template
new file:   boardfont.svg
new file:   img/00101P3.png
new file:   mainboard/apple1template.kicad_wks
additional work on mainboard
Parts:
- C31: footprint mainboard:apple-1_CP_5300UF_15V_+- -> mainboard:CP_Axial_5300uF
Other:
- title: Apple I - Power Supply -> Processor Section
Changed lines of the file:
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@@
 	(paper "A4")
 	(title_block
-		(title "Apple I - Power Supply")
+		(title "Processor Section")
 		(date "2019-08-11")
 		(comment 1 "Drawn by Nicolas Robin")
@@
 	)
 	(symbol
+		(lib_name "CP1_1")
 		(lib_id "Device:CP1")
 		(at 124.46 57.15 0)
@@
 			)
 		)
-		(property "Footprint" "mainboard:apple-1_CP_5300UF_15V_+-"
+		(property "Footprint" "mainboard:CP_Axial_5300uF"
 			(at 124.46 57.15 0)
 			(hide yes)

Commit message: board is now complete, cleanup work can begin
Other:
- title: Processor Section -> Apple I - Processor Section
Changed lines of the file:
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@@
 	(paper "A4")
 	(title_block
-		(title "Processor Section")
+		(title "Apple I - Processor Section")
 		(date "2019-08-11")
 		(comment 1 "Drawn by Nicolas Robin")
