File: mainboard/transformers.kicad_sch (KiCad schematic)
At the start: 6 parts, among them J1 Conn_01x06, P1 Conn_WallPlug_Earth, SW1 ON/OFF, T1 STANCOR P-8380, T2 STANCOR P-8667

Commit message: merged /transformers with /mainboard
Parts:
- J15: renamed from J1; now not fitted
- P1, SW1: now left out of the parts list
- T1, T2: symbol apple1_transformers:Transformer -> apple1:Transformer
Connections:
- net at T1.~: now also J15.2 (Pin_2)
- new net: SW1.2 (B), T1.~, T2.~
- new net: F1.1, T1.~, T2.~
Other:
- title: Apple I - AC Power Supply -> (none)
- moved on the sheet: T1, T2

Commit message: mainboard work
Parts:
- J15: now fitted
- P1: now not fitted
Connections:
- net at T1.~: now also J15.2 (Pin_2)
- new net: SW1.2 (B), T1.~, T2.~
- new net: F1.1, T1.~, T2.~
Changed lines of the file:
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@@
 		(on_board no)
 		(in_pos_files yes)
-		(dnp no)
+		(dnp yes)
 		(property "Reference" "P1"
 			(at 66.675 75.565 0)
@@
 		(on_board no)
 		(in_pos_files yes)
-		(dnp yes)
+		(dnp no)
 		(property "Reference" "J15"
 			(at 160.782 97.8916 0)

Commit message: added kicad drawing template
new file:   boardfont.svg
new file:   img/00101P3.png
new file:   mainboard/apple1template.kicad_wks
additional work on mainboard
Connections:
- net at T1.~: now also J15.2 (Pin_2)
- new net: SW1.2 (B), T1.~, T2.~
- new net: F1.1, T1.~, T2.~
Other:
- title: (none) -> Processor Section
Changed lines of the file:
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@@
 	(generator_version "10.0")
 	(paper "A")
+	(title_block
+		(title "Processor Section")
+		(comment 1 "Drawn by Nicolas Robin")
+	)
 	(text "10V C.T."
 		(exclude_from_sim no)

Commit message: board is now complete, cleanup work can begin
Connections:
- net at T1.~: now also J15.2 (Pin_2)
- new net: SW1.2 (B), T1.~, T2.~
- new net: F1.1, T1.~, T2.~
Other:
- title: Processor Section -> Apple I - Processor Section
Changed lines of the file:
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@@
 	(paper "A")
 	(title_block
-		(title "Processor Section")
+		(title "Apple I - Processor Section")
 		(comment 1 "Drawn by Nicolas Robin")
 	)
