File: aci/aci.kicad_sch (KiCad schematic)
At the start: 23 parts, among them J1 Switchcraft #41, J2 Switchcraft #41, J3 ACI_EdgeConnector, Q1 Q_NPN_EBC, Q2 Q_NPN_EBC

Commit message: new file:   aci/README.md modified:   aci/aci.kicad_pcb new file:   aci/aci.kicad_pro modified:   aci/aci.kicad_sch deleted:    aci/aci.pro deleted:    aci/aci.sch new file:   doc/apple1cassette.pdf deleted:    doc/progress3d.png
Parts:
- A1: footprint ~ -> Package_DIP:DIP-8_W7.62mm
- A2, A5, A6: footprint ~ -> Package_DIP:DIP-14_W7.62mm
- A3, A4: footprint ~ -> Package_DIP:DIP-16_W7.62mm
- D1: footprint ~ -> LED_THT:LED_D4.0mm
- J1, J2: footprint ~ -> (none)
- Q1, Q2: footprint ~ -> Package_TO_SOT_THT:TO-92
- R1, R10, R2, R3, R4, R5, R6, R7, R8, R9: footprint ~ -> Resistor_THT:R_Axial_DIN0207_L6.3mm_D2.5mm_P10.16mm_Horizontal
Changed lines of the file:
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@@
 			)
 		)
-		(property "Footprint" "~"
+		(property "Footprint" "Package_DIP:DIP-8_W7.62mm"
 			(at 109.22 121.92 0)
 			(hide yes)
@@
 			)
 		)
-		(property "Datasheet" "~"
+		(property "Datasheet" "https://www.ti.com/lit/ds/symlink/lm311.pdf?ts=1780338572961"
 			(at 109.22 121.92 0)
 			(hide yes)
@@
 			)
 		)
-		(property "Footprint" "~"
+		(property "Footprint" "Package_DIP:DIP-14_W7.62mm"
 			(at 144.78 43.18 0)
 			(hide yes)
@@
 			)
 		)
-		(property "Datasheet" "~"
+		(property "Datasheet" "https://www.ti.com/lit/ds/symlink/sn74ls74a.pdf?ts=1780318698351"
 			(at 144.78 43.18 0)
 			(hide yes)
@@
 			)
 		)
-		(property "Footprint" "~"
+		(property "Footprint" "Package_DIP:DIP-14_W7.62mm"
 			(at 76.2 38.1 0)
 			(hide yes)
@@
 			)
 		)
-		(property "Datasheet" "~"
+		(property "Datasheet" "https://www.ti.com/lit/ds/symlink/sn74ls02.pdf"
 			(at 76.2 38.1 0)
 			(hide yes)
@@
 			)
 		)
-		(property "Footprint" "~"
+		(property "Footprint" "Package_DIP:DIP-14_W7.62mm"
 			(at 99.06 40.64 0)
 			(hide yes)
@@
 			)
 		)
-		(property "Datasheet" "~"
+		(property "Datasheet" "https://www.ti.com/lit/ds/symlink/sn74ls10.pdf?ts=1780308043680"
 			(at 99.06 40.64 0)
 			(hide yes)
@@
 			)
 		)
-		(property "Footprint" "~"
+		(property "Footprint" "Package_DIP:DIP-16_W7.62mm"
 			(at 205.74 119.38 0)
 			(hide yes)
@@
 			)
 		)
-		(property "Datasheet" "~"
+		(property "Datasheet" "https://datasheet4u.com/pdf/1560877/82S129.pdf"
 			(at 205.74 119.38 0)
 			(hide yes)
@@
 			)
 		)
-		(property "Footprint" "~"
+		(property "Footprint" "Package_DIP:DIP-14_W7.62mm"
 			(at 76.2 53.34 0)
 			(hide yes)
@@
 			)
 		)
-		(property "Datasheet" "~"
+		(property "Datasheet" "https://www.ti.com/lit/ds/symlink/sn74ls02.pdf"
 			(at 76.2 53.34 0)
 			(hide yes)
@@
 			)
 		)
-		(property "Footprint" "~"
+		(property "Footprint" "Package_DIP:DIP-14_W7.62mm"
 			(at 121.92 43.18 0)
 			(hide yes)
@@
 			)
 		)
-		(property "Datasheet" "~"
+		(property "Datasheet" "https://www.ti.com/lit/ds/symlink/sn74ls02.pdf"
 			(at 121.92 43.18 0)
 			(hide yes)
@@
 			)
 		)
-		(property "Footprint" "~"
+		(property "Footprint" "Package_DIP:DIP-14_W7.62mm"
 			(at 144.78 78.74 0)
 			(hide yes)
@@
 			)
 		)
-		(property "Datasheet" "~"
+		(property "Datasheet" "https://www.ti.com/lit/ds/symlink/sn74ls10.pdf?ts=1780308043680"
 			(at 144.78 78.74 0)
 			(hide yes)
@@
 			)
 		)
-		(property "Footprint" "~"
+		(property "Footprint" "Package_DIP:DIP-14_W7.62mm"
 			(at 167.64 81.28 0)
 			(hide yes)
@@
 			)
 		)
-		(property "Datasheet" "~"
+		(property "Datasheet" "https://www.ti.com/lit/ds/symlink/sn74ls10.pdf?ts=1780308043680"
 			(at 167.64 81.28 0)
 			(hide yes)
@@
 			)
 		)
-		(property "Footprint" "~"
+		(property "Footprint" "Package_DIP:DIP-14_W7.62mm"
 			(at 190.5 81.28 0)
 			(hide yes)
@@
 			)
 		)
-		(property "Datasheet" "~"
+		(property "Datasheet" "https://www.ti.com/lit/ds/symlink/sn74ls02.pdf"
 			(at 190.5 81.28 0)
 			(hide yes)
@@
 			)
 		)
-		(property "Footprint" "~"
+		(property "Footprint" "Package_DIP:DIP-16_W7.62mm"
 			(at 254 119.38 0)
 			(hide yes)
@@
 			)
 		)
-		(property "Datasheet" "~"
+		(property "Datasheet" "https://datasheet4u.com/pdf/1560877/82S129.pdf"
 			(at 254 119.38 0)
 			(hide yes)
@@
 			)
 		)
-		(property "Footprint" "~"
+		(property "Footprint" "Package_TO_SOT_THT:TO-92"
 			(at 88.9 167.64 0)
 			(hide yes)
@@
 			)
 		)
-		(property "Footprint" "~"
+		(property "Footprint" "Package_TO_SOT_THT:TO-92"
 			(at 96.52 172.72 0)
 			(hide yes)
@@
 			)
 		)
-		(property "Footprint" "~"
+		(property "Footprint" "Resistor_THT:R_Axial_DIN0207_L6.3mm_D2.5mm_P10.16mm_Horizontal"
 			(at 76.2 170.18 0)
 			(hide yes)
@@
 			)
 		)
-		(property "Footprint" "~"
+		(property "Footprint" "Resistor_THT:R_Axial_DIN0207_L6.3mm_D2.5mm_P10.16mm_Horizontal"
 			(at 93.98 157.48 0)
 			(hide yes)
@@
 			)
 		)
-		(property "Footprint" "~"
+		(property "Footprint" "LED_THT:LED_D4.0mm"
 			(at 93.98 162.56 90)
 			(hide yes)
@@
 			)
 		)
-		(property "Footprint" "~"
+		(property "Footprint" ""
 			(at 58.42 124.46 0)
 			(hide yes)
@@
 			)
 		)
-		(property "Footprint" "~"
+		(property "Footprint" ""
 			(at 177.8 50.8 0)
 			(hide yes)
@@
 			)
 		)
-		(property "Footprint" "~"
+		(property "Footprint" "Resistor_THT:R_Axial_DIN0207_L6.3mm_D2.5mm_P10.16mm_Horizontal"
 			(at 81.28 114.3 0)
 			(hide yes)
@@
 			)
 		)
-		(property "Footprint" "~"
+		(property "Footprint" "Resistor_THT:R_Axial_DIN0207_L6.3mm_D2.5mm_P10.16mm_Horizontal"
 			(at 91.44 114.3 0)
 			(hide yes)
@@
 			)
 		)
-		(property "Footprint" "~"
+		(property "Footprint" "Resistor_THT:R_Axial_DIN0207_L6.3mm_D2.5mm_P10.16mm_Horizontal"
 			(at 81.28 129.54 0)
 			(hide yes)
@@
 			)
 		)
-		(property "Footprint" "~"
+		(property "Footprint" "Resistor_THT:R_Axial_DIN0207_L6.3mm_D2.5mm_P10.16mm_Horizontal"
 			(at 91.44 129.54 0)
 			(hide yes)
@@
 			)
 		)
-		(property "Footprint" "~"
+		(property "Footprint" "Resistor_THT:R_Axial_DIN0207_L6.3mm_D2.5mm_P10.16mm_Horizontal"
 			(at 119.38 116.84 0)
 			(hide yes)
@@
 			)
 		)
-		(property "Footprint" "~"
+		(property "Footprint" "Resistor_THT:R_Axial_DIN0207_L6.3mm_D2.5mm_P10.16mm_Horizontal"
 			(at 119.38 127 0)
 			(hide yes)
@@
 			)
 		)
-		(property "Footprint" "~"
+		(property "Footprint" "Resistor_THT:R_Axial_DIN0207_L6.3mm_D2.5mm_P10.16mm_Horizontal"
 			(at 162.56 45.72 0)
 			(hide yes)
@@
 			)
 		)
-		(property "Footprint" "~"
+		(property "Footprint" "Resistor_THT:R_Axial_DIN0207_L6.3mm_D2.5mm_P10.16mm_Horizontal"
 			(at 162.56 55.88 0)
 			(hide yes)
@@
 			)
 		)
-		(property "Footprint" "~"
+		(property "Footprint" "Package_DIP:DIP-14_W7.62mm"
 			(at 220.98 48.26 0)
 			(hide yes)
@@
 			)
 		)
-		(property "Datasheet" "~"
+		(property "Datasheet" "https://www.ti.com/lit/ds/symlink/sn74ls74a.pdf?ts=1780318698351"
 			(at 220.98 48.26 0)
 			(hide yes)
@@
 			)
 		)
-		(property "Footprint" "~"
+		(property "Footprint" "Package_DIP:DIP-14_W7.62mm"
 			(at 233.68 48.26 0)
 			(hide yes)
@@
 			)
 		)
-		(property "Datasheet" "~"
+		(property "Datasheet" "https://www.ti.com/lit/ds/symlink/sn74ls02.pdf"
 			(at 233.68 48.26 0)
 			(hide yes)
@@
 			)
 		)
-		(property "Footprint" "~"
+		(property "Footprint" "Package_DIP:DIP-14_W7.62mm"
 			(at 246.38 48.26 0)
 			(hide yes)
@@
 			)
 		)
-		(property "Datasheet" "~"
+		(property "Datasheet" "https://www.ti.com/lit/ds/symlink/sn74ls10.pdf?ts=1780308043680"
 			(at 246.38 48.26 0)
 			(hide yes)

Commit message: modified:   aci/README.md 	modified:   aci/aci.kicad_pcb 	modified:   aci/aci.kicad_sch 	new file:   aci/aci.pretty/aci_TO-92_bent.kicad_mod 	new file:   aci/fp-lib-table 	new file:   doc/aci-assembly-v0.18.pdf 	modified:   mainboard/mainboard.kicad_pcb 	modified:   mainboard/mainboard.kicad_pro
Parts:
- Q1, Q2: footprint Package_TO_SOT_THT:TO-92 -> aci:aci_TO-92_bent
Changed lines of the file:
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@@
 			)
 		)
-		(property "Footprint" "Package_TO_SOT_THT:TO-92"
+		(property "Footprint" "aci:aci_TO-92_bent"
 			(at 88.9 167.64 0)
 			(hide yes)
@@
 			)
 		)
-		(property "Footprint" "Package_TO_SOT_THT:TO-92"
+		(property "Footprint" "aci:aci_TO-92_bent"
 			(at 96.52 172.72 0)
 			(hide yes)
