File: aci/aci.kicad_sch (KiCad schematic)
At the start: 23 parts, among them J1 Switchcraft #41, J2 Switchcraft #41, J3 ACI_EdgeConnector, Q1 Q_NPN_EBC, Q2 Q_NPN_EBC

Commit message: additional footprint work
Parts:
- A1: footprint Package_DIP:DIP-8_W7.62mm -> aci:apple-1_DIP-8_W7.62mm
- A2, A5, A6: footprint Package_DIP:DIP-14_W7.62mm -> aci:apple-1_DIP-14_W7.62mm
- A3, A4: footprint Package_DIP:DIP-16_W7.62mm -> aci:apple-1_DIP-16_W7.62mm
Changed lines of the file:
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@@
 			)
 		)
-		(property "Footprint" "Package_DIP:DIP-8_W7.62mm"
+		(property "Footprint" "aci:apple-1_DIP-8_W7.62mm"
 			(at 109.22 121.92 0)
 			(hide yes)
@@
 			)
 		)
-		(property "Footprint" "Package_DIP:DIP-14_W7.62mm"
+		(property "Footprint" "aci:apple-1_DIP-14_W7.62mm"
 			(at 144.78 43.18 0)
 			(hide yes)
@@
 			)
 		)
-		(property "Footprint" "Package_DIP:DIP-14_W7.62mm"
+		(property "Footprint" "aci:apple-1_DIP-14_W7.62mm"
 			(at 76.2 38.1 0)
 			(hide yes)
@@
 			)
 		)
-		(property "Footprint" "Package_DIP:DIP-14_W7.62mm"
+		(property "Footprint" "aci:apple-1_DIP-14_W7.62mm"
 			(at 99.06 40.64 0)
 			(hide yes)
@@
 			)
 		)
-		(property "Footprint" "Package_DIP:DIP-16_W7.62mm"
+		(property "Footprint" "aci:apple-1_DIP-16_W7.62mm"
 			(at 205.74 119.38 0)
 			(hide yes)
@@
 			)
 		)
-		(property "Footprint" "Package_DIP:DIP-14_W7.62mm"
+		(property "Footprint" "aci:apple-1_DIP-14_W7.62mm"
 			(at 76.2 53.34 0)
 			(hide yes)
@@
 			)
 		)
-		(property "Footprint" "Package_DIP:DIP-14_W7.62mm"
+		(property "Footprint" "aci:apple-1_DIP-14_W7.62mm"
 			(at 121.92 43.18 0)
 			(hide yes)
@@
 			)
 		)
-		(property "Footprint" "Package_DIP:DIP-14_W7.62mm"
+		(property "Footprint" "aci:apple-1_DIP-14_W7.62mm"
 			(at 144.78 78.74 0)
 			(hide yes)
@@
 			)
 		)
-		(property "Footprint" "Package_DIP:DIP-14_W7.62mm"
+		(property "Footprint" "aci:apple-1_DIP-14_W7.62mm"
 			(at 167.64 81.28 0)
 			(hide yes)
@@
 			)
 		)
-		(property "Footprint" "Package_DIP:DIP-14_W7.62mm"
+		(property "Footprint" "aci:apple-1_DIP-14_W7.62mm"
 			(at 190.5 81.28 0)
 			(hide yes)
@@
 			)
 		)
-		(property "Footprint" "Package_DIP:DIP-16_W7.62mm"
+		(property "Footprint" "aci:apple-1_DIP-16_W7.62mm"
 			(at 254 119.38 0)
 			(hide yes)
@@
 			)
 		)
-		(property "Footprint" "Package_DIP:DIP-14_W7.62mm"
+		(property "Footprint" "aci:apple-1_DIP-14_W7.62mm"
 			(at 220.98 48.26 0)
 			(hide yes)
@@
 			)
 		)
-		(property "Footprint" "Package_DIP:DIP-14_W7.62mm"
+		(property "Footprint" "aci:apple-1_DIP-14_W7.62mm"
 			(at 233.68 48.26 0)
 			(hide yes)
@@
 			)
 		)
-		(property "Footprint" "Package_DIP:DIP-14_W7.62mm"
+		(property "Footprint" "aci:apple-1_DIP-14_W7.62mm"
 			(at 246.38 48.26 0)
 			(hide yes)

Commit message: completed aci, added p-l4b boards
Parts:
- C1: footprint ~ -> aci:C_Disc_.01_p350MILS
- J1: footprint (none) -> aci:aci_phonopads_frmtape
- J2: footprint (none) -> aci:aci_phonopads
- J3: footprint ~ -> aci:aci_edgecon
- R1, R10, R2, R3, R4, R5, R6, R7, R8, R9: footprint Resistor_THT:R_Axial_DIN0207_L6.3mm_D2.5mm_P10.16mm_Horizontal -> aci:R_Axial_ACI
Changed lines of the file:
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@@
 			)
 		)
-		(property "Footprint" "Resistor_THT:R_Axial_DIN0207_L6.3mm_D2.5mm_P10.16mm_Horizontal"
+		(property "Footprint" "aci:R_Axial_ACI"
 			(at 76.2 170.18 0)
 			(hide yes)
@@
 			)
 		)
-		(property "Footprint" "Resistor_THT:R_Axial_DIN0207_L6.3mm_D2.5mm_P10.16mm_Horizontal"
+		(property "Footprint" "aci:R_Axial_ACI"
 			(at 93.98 157.48 0)
 			(hide yes)
@@
 			)
 		)
-		(property "Footprint" ""
+		(property "Footprint" "aci:aci_phonopads_frmtape"
 			(at 58.42 124.46 0)
 			(hide yes)
@@
 			)
 		)
-		(property "Footprint" ""
+		(property "Footprint" "aci:aci_phonopads"
 			(at 177.8 50.8 0)
 			(hide yes)
@@
 			)
 		)
-		(property "Footprint" "Resistor_THT:R_Axial_DIN0207_L6.3mm_D2.5mm_P10.16mm_Horizontal"
+		(property "Footprint" "aci:R_Axial_ACI"
 			(at 81.28 114.3 0)
 			(hide yes)
@@
 			)
 		)
-		(property "Footprint" "Resistor_THT:R_Axial_DIN0207_L6.3mm_D2.5mm_P10.16mm_Horizontal"
+		(property "Footprint" "aci:R_Axial_ACI"
 			(at 91.44 114.3 0)
 			(hide yes)
@@
 			)
 		)
-		(property "Footprint" "Resistor_THT:R_Axial_DIN0207_L6.3mm_D2.5mm_P10.16mm_Horizontal"
+		(property "Footprint" "aci:R_Axial_ACI"
 			(at 81.28 129.54 0)
 			(hide yes)
@@
 			)
 		)
-		(property "Footprint" "Resistor_THT:R_Axial_DIN0207_L6.3mm_D2.5mm_P10.16mm_Horizontal"
+		(property "Footprint" "aci:R_Axial_ACI"
 			(at 91.44 129.54 0)
 			(hide yes)
@@
 			)
 		)
-		(property "Footprint" "Resistor_THT:R_Axial_DIN0207_L6.3mm_D2.5mm_P10.16mm_Horizontal"
+		(property "Footprint" "aci:R_Axial_ACI"
 			(at 119.38 116.84 0)
 			(hide yes)
@@
 			)
 		)
-		(property "Footprint" "Resistor_THT:R_Axial_DIN0207_L6.3mm_D2.5mm_P10.16mm_Horizontal"
+		(property "Footprint" "aci:R_Axial_ACI"
 			(at 119.38 127 0)
 			(hide yes)
@@
 			)
 		)
-		(property "Footprint" "~"
+		(property "Footprint" "aci:C_Disc_.01_p350MILS"
 			(at 76.2 124.46 0)
 			(hide yes)
@@
 			)
 		)
-		(property "Footprint" "~"
+		(property "Footprint" "aci:aci_edgecon"
 			(at 62.23 58.42 0)
 			(hide yes)
@@
 			)
 		)
-		(property "Footprint" "~"
+		(property "Footprint" "aci:aci_edgecon"
 			(at 62.23 83.82 0)
 			(hide yes)
@@
 			)
 		)
-		(property "Footprint" "~"
+		(property "Footprint" "aci:aci_edgecon"
 			(at 220.98 130.81 0)
 			(hide yes)
@@
 			)
 		)
-		(property "Footprint" "Resistor_THT:R_Axial_DIN0207_L6.3mm_D2.5mm_P10.16mm_Horizontal"
+		(property "Footprint" "aci:R_Axial_ACI"
 			(at 162.56 45.72 0)
 			(hide yes)
@@
 			)
 		)
-		(property "Footprint" "Resistor_THT:R_Axial_DIN0207_L6.3mm_D2.5mm_P10.16mm_Horizontal"
+		(property "Footprint" "aci:R_Axial_ACI"
 			(at 162.56 55.88 0)
 			(hide yes)

Commit message: merged /transformers with /mainboard
Parts:
- added C2, C3: .1UF, aci:C_AxialDecoupling, symbol Device:C
- C1: value 0.01u -> 0.01UF
Connections:
- net +5V: now also C2.1, C3.1
- net GND: now also C2.2, C3.2
