File: serialboard/serialboard.kicad_pcb (KiCad board)
At the start: 2 copper layers, 162.8 x 77.7 mm, 0 parts

Commit message: completed aci, added p-l4b boards
Parts:
- added U1: L7805, Package_TO_SOT_THT:TO-220-3_Horizontal_TabDown, F.Cu at (186.7, 55.1)
- added U2: KM28C64A, Package_DIP:DIP-28_W15.24mm_Socket_LongPads, F.Cu at (171.7, 85.1)
- added U3: 74LS257, Package_DIP:DIP-16_W7.62mm_Socket_LongPads, F.Cu at (114.8, 104.4)
- added U4: 74LS257, Package_DIP:DIP-16_W7.62mm_Socket_LongPads, F.Cu at (138.9, 104.4)
- added U5: ATmega328P-P, Package_DIP:DIP-28_W7.62mm_Socket_LongPads, F.Cu at (98.0, 71.4)
- added U6: 7402, Package_DIP:DIP-14_W7.62mm_Socket_LongPads, F.Cu at (128.0, 61.2)
- added U7: LM358, Package_DIP:DIP-8_W7.62mm_Socket_LongPads, F.Cu at (84.3, 79.0)
- added U8: MAX232, Package_DIP:DIP-16_W7.62mm_Socket_LongPads, F.Cu at (54.3, 102.0)
Routing:
- net (no net): track 5174.0 -> 599.9 mm, vias 309 -> 40
- net Net-(U5-GND-Pad22): track 0.00 -> 672.6 mm, vias 0 -> 25
- net unconnected-(U5-VCC-Pad7): track 0.00 -> 482.6 mm, vias 0 -> 27
- net unconnected-(U5-PB0-Pad14): track 0.00 -> 217.1 mm, vias 0 -> 3
- net unconnected-(U5-PD7-Pad13): track 0.00 -> 208.2 mm, vias 0 -> 3
- net unconnected-(U6-Pad2): track 0.00 -> 178.2 mm, vias 0 -> 4
- net unconnected-(U2-I/O7-Pad19): track 0.00 -> 131.9 mm, vias 0 -> 2
- net unconnected-(U2-I/O6-Pad18): track 0.00 -> 131.6 mm, vias 0 -> 2
- net unconnected-(U2-I/O5-Pad17): track 0.00 -> 125.0 mm, vias 0 -> 1
- net unconnected-(U2-I/O4-Pad16): track 0.00 -> 121.7 mm, vias 0 -> 2
- net unconnected-(U2-I/O3-Pad15): track 0.00 -> 108.9 mm, vias 0 -> 1
- net unconnected-(U2-I/O2-Pad13): track 0.00 -> 101.6 mm, vias 0 -> 2
- net unconnected-(U5-PB1-Pad15): track 0.00 -> 101.0 mm, vias 0 -> 1
- net unconnected-(U1-IN-Pad1): track 0.00 -> 97.6 mm, vias 0 -> 3
- net unconnected-(U2-I/O0-Pad11): track 0.00 -> 97.6 mm, vias 0 -> 3
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