File: serialboard/serialboard.kicad_sch (KiCad schematic)
At the start: 0 parts

Commit message: completed aci, added p-l4b boards
Parts:
- added U1: L7805, Package_TO_SOT_THT:TO-220-3_Horizontal_TabDown, symbol Regulator_Linear:L7805
- added U2: KM28C64A, Package_DIP:DIP-28_W15.24mm_Socket_LongPads, symbol Memory_EEPROM:KM28C64A
- added U3, U4: 74LS257, Package_DIP:DIP-16_W7.62mm_Socket_LongPads, symbol 74xx:74LS257
- added U5: ATmega328P-P, Package_DIP:DIP-28_W7.62mm_Socket_LongPads, symbol MCU_Microchip_ATmega:ATmega328P-P
- added U6: 7402, Package_DIP:DIP-14_W7.62mm_Socket_LongPads, symbol 74xx:7402
- added U7: LM358, Package_DIP:DIP-8_W7.62mm_Socket_LongPads, symbol Amplifier_Operational:LM358
- added U8: MAX232, Package_DIP:DIP-16_W7.62mm_Socket_LongPads, symbol Interface_UART:MAX232
Connections:
- new net: U5.22 (GND), U5.8 (GND)
