File: datanetics_modern/datanetics_modern.kicad_pcb (KiCad board)
At the start: 2 copper layers, 298.4 x 139.7 mm, 169 parts, among them J1 CONN_2X15_LINEAR_ALPHA, P1 jumper_pth, P10 jumper_pth, P11 jumper_pth, P12 jumper_pth, P13 jumper_pth, P14 jumper_pth, P15 jumper_pth, P16 jumper_pth, P17 jumper_pth, P18 jumper_pth, P19 jumper_pth, P2 jumper_pth, P20 jumper_pth, P21 jumper_pth, P22 jumper_pth, P23 jumper_pth, P24 jumper_pth, P25 jumper_pth, P26 jumper_pth, P27 jumper_pth, P28 jumper_pth, P29 jumper_pth, P3 jumper_pth, P30 jumper_pth, P31 jumper_pth, P32 jumper_pth, P33 jumper_pth, P34 jumper_pth, P35 jumper_pth, P36 jumper_pth, P37 jumper_pth, P38 jumper_pth, P39 jumper_pth, P4 jumper_pth, P40 jumper_pth, P41 jumper_pth, P42 jumper_pth, P43 jumper_pth, P44 jumper_pth, P45 jumper_pth, P46 jumper_pth, P47 jumper_pth, P48 jumper_pth, P49 jumper_pth, P5 jumper_pth, P50 jumper_pth, P51 jumper_pth, P52 jumper_pth, P53 jumper_pth, P54 jumper_pth, P55 jumper_pth, P56 jumper_pth, P57 jumper_pth, P58 jumper_pth, P59 jumper_pth, P6 jumper_pth, P60 jumper_pth, P61 jumper_pth, P62 jumper_pth, P63 jumper_pth, P64 jumper_pth, P65 jumper_pth, P66 jumper_pth, P67 jumper_pth, P68 jumper_pth, P69 jumper_pth, P7 jumper_pth, P70 jumper_pth, P71 jumper_pth, P72 jumper_pth, P73 jumper_pth, P74 jumper_pth, P75 jumper_pth, P76 jumper_pth, P8 jumper_pth, P9 jumper_pth, SW1 RESET, SW10 LF, SW11 P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

Commit message: additional footprint refinement and mainboard update
Parts:
- SW1, SW10, SW11, SW12, SW13, SW14, SW15, SW16, SW17, SW18, SW19, SW2, SW20, SW21, SW22, SW23, SW24, SW25, SW26, SW27, SW28, SW29, SW3, SW30, SW31, SW32, SW33, SW34, SW35, SW36, SW37, SW38, SW39, SW4, SW40, SW41, SW42, SW43, SW44, SW45, SW46, SW47, SW48, SW49, SW5, SW50, SW51, SW52, SW53, SW54, SW55, SW56, SW6, SW7, SW9: footprint PCM_Switch_Keyboard_Cherry_MX:SW_Cherry_MX_PCB -> datanetics_modern:dn_SW_Cherry_MX_PCB
- SW8: footprint PCM_Switch_Keyboard_Cherry_MX:SW_Cherry_MX_PCB -> datanetics_modern:dn_SW_Cherry_MX_PCB_SPACEBAR
- U1: footprint Package_DIP:DIP-40_W15.24mm -> datanetics_modern:dn_DIP-40_W15.24mm
Other:
- board text added: "2) SILKSCREEN LAYER PRESENT BUT NOT TO BE APPLIED 1) DO NOT APPLY SOLDERMASK TO PART FABRICATION NOTES:"
- board text added: "EDGE CONNECTOR TO BE PLATED IN HARD GOLD WITHIN THE HATCHED ZONE SHOWN"
- board text removed: "Replica © 2022 Tube Time After Mike Willegal's replica"

Commit message: mainboard work
Parts:
- added REF**: Stabilizer_Cherry_MX_7.00u, PCM_Mounting_Keyboard_Stabilizer:Stabilizer_Cherry_MX_7.00u, F.Cu at (189.9, 190.5)
- added REF**: Stabilizer_Cherry_MX_8.00u, PCM_Mounting_Keyboard_Stabilizer:Stabilizer_Cherry_MX_8.00u, F.Cu at (189.9, 190.5)
- U1: footprint datanetics_modern:dn_DIP-40_W15.24mm -> Package_DIP:DIP-40_W15.24mm
